Commit message: new branch

File: src/robot_description/urdf/ur5.urdf.xacro (robot description, xacro)
@@ -27,5 +27,5 @@
     center_of_mass = [ [0, -0.02561, 0.00193], [0.2125, 0, 0.11336], [0.11993, 0.0, 0.0265], [0, -0.0018, 0.01634], [0, 0.0018,0.01634], [0, 0, -0.001159] ]
   -->
-  <xacro:property name="ur5_d1" value="0.089159" />
+  <xacro:property name="ur5_d1" value="0.165" />
   <xacro:property name="ur5_a2" value="-0.42500" />
   <xacro:property name="ur5_a3" value="-0.39225" />
